File: can_servo_x6_breakout/can_servo_x6_breakout.sch (KiCad schematic (older format))
At the start: 8 parts, among them J1 CAN_SERVO, J2 CAN_SERVO, J3 CAN_PIXHAWK, J4 CAN_SERVO, J5 V_IN

Commit message: Added a ground plane where it was forgotten
Parts:
- AFA1: symbol ARCL:afa_logo -> can_servo_x6_breakout-rescue:afa_logo-ARCL
Changed lines of the file:
@@
 	5850 1350 5950 1350
 $Comp
-L ARCL:afa_logo AFA1
+L can_servo_x6_breakout-rescue:afa_logo-ARCL AFA1
 U 1 1 5F693BDA
 P 4350 3650
