File: i2c_breakout/i2c_breakout.sch (KiCad schematic (older format))
At the start: 8 parts, among them J1 Conn_01x02_Male, J2 Conn_01x04_Male, J3 Conn_01x04_Male, J4 Conn_01x04_Male, J5 Conn_01x04_Male, J6 Conn_01x04_Male, J7 5V, J8 GND

Commit message: Added a ground plane where it was forgotten
Parts:
- J1: value Conn_01x02_Male -> Conn_01x04_Male; footprint Connector_JST:JST_GH_BM02B-GHS-TBT_1x02-1MP_P1.25mm_Vertical -> Connector_JST:JST_GH_BM04B-GHS-TBT_1x04-1MP_P1.25mm_Vertical; symbol Connector:Conn_01x02_Male -> Connector:Conn_01x04_Male
Connections:
- net Earth: now also J1.4 (Pin_4); no longer J1.2 (Pin_2)
- net at J2.2 (Pin_2), J3.2 (Pin_2), J4.2 (Pin_2)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: now also J1.2 (Pin_2)
- net at J2.3 (Pin_3), J3.3 (Pin_3), J4.3 (Pin_3)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: now also J1.3 (Pin_3)
Changed lines of the file:
@@
 $EndComp
 $Comp
-L Connector:Conn_01x02_Male J1
+L Connector:Conn_01x04_Male J1
 U 1 1 616CEFDD
-P 5100 2450
-F 0 "J1" H 5208 2631 50  0000 C CNN
-F 1 "Conn_01x02_Male" H 5208 2540 50  0000 C CNN
-F 2 "Connector_JST:JST_GH_BM02B-GHS-TBT_1x02-1MP_P1.25mm_Vertical" H 5100 2450 50  0001 C CNN
-F 3 "~" H 5100 2450 50  0001 C CNN
-	1    5100 2450
+P 5800 2450
+F 0 "J1" H 5950 2700 50  0000 C CNN
+F 1 "Conn_01x04_Male" H 5900 2650 50  0000 C CNN
+F 2 "Connector_JST:JST_GH_BM04B-GHS-TBT_1x04-1MP_P1.25mm_Vertical" H 5800 2450 50  0001 C CNN
+F 3 "~" H 5800 2450 50  0001 C CNN
+	1    5800 2450
 	1    0    0    -1
 $EndComp
-Wire Wire Line
-	5300 2450 5650 2450
-Wire Wire Line
-	5650 2450 5650 2350
-Wire Wire Line
-	5650 2350 5800 2350
 Connection ~ 6350 2350
 Wire Wire Line
@@
 Wire Wire Line
 	7000 2350 7300 2350
-Wire Wire Line
-	5300 2550 5650 2550
-Wire Wire Line
-	5650 2550 5650 2650
-Wire Wire Line
-	5650 2650 5800 2650
 Connection ~ 6350 2650
 Wire Wire Line
@@
 Wire Wire Line
 	5800 2350 5800 2100
-Connection ~ 5800 2350
 Wire Wire Line
-	5800 2350 6350 2350
+	5800 2350 6000 2350
 Wire Wire Line
 	5800 2650 5800 2800
-Connection ~ 5800 2650
 Wire Wire Line
-	5800 2650 6350 2650
+	5800 2650 6000 2650
 $Comp
 L Connector:Conn_01x01_Male J7
@@
 	1    0    0    -1
 $EndComp
+Connection ~ 6000 2350
+Wire Wire Line
+	6000 2350 6350 2350
+Connection ~ 6000 2650
+Wire Wire Line
+	6000 2650 6350 2650
+Wire Wire Line
+	6000 2450 6350 2450
+Connection ~ 6350 2450
+Wire Wire Line
+	6350 2550 6000 2550
+Connection ~ 6350 2550
 $EndSCHEMATC
