File: gps_i2c_breakout/gps_i2c_breakout.sch (KiCad schematic (older format))
At the start: 7 parts, among them J1 Conn_01x02_Male, J2 Conn_01x04_Male, J3 Conn_01x04_Male, J4 Conn_01x04_Male, J5 Conn_01x04_Male, J7 5V, J8 GND

Commit message: Updated the I2C and GPS breakout boards with ground fills
Parts:
- removed J1: Conn_01x02_Male, Connector_JST:JST_GH_BM02B-GHS-TBT_1x02-1MP_P1.25mm_Vertical, symbol Connector:Conn_01x02_Male
- added J6: Conn_01x06_Male, Connector_JST:JST_GH_BM06B-GHS-TBT_1x06-1MP_P1.25mm_Vertical, symbol Connector:Conn_01x06_Male
- J4: footprint Connector_JST:JST_GH_BM06B-GHS-TBT_1x06-1MP_P1.25mm_Vertical -> Connector_JST:JST_GH_BM04B-GHS-TBT_1x04-1MP_P1.25mm_Vertical; symbol Connector:Conn_01x06_Male -> Connector:Conn_01x04_Male
- J5: value Conn_01x04_Male -> Conn_01x06_Male
Connections:
- net +5V: now also J6.1 (Pin_1)
- net Earth: now also J4.4 (Pin_4), J6.6 (Pin_6); no longer J4.6 (Pin_6)
- net at J2.2 (Pin_2), J3.2 (Pin_2), J5.4 (Pin_4): now also J4.2 (Pin_2), J6.4 (Pin_4); no longer J4.4 (Pin_4)
- net at J2.3 (Pin_3), J3.3 (Pin_3), J5.5 (Pin_5): now also J4.3 (Pin_3), J6.5 (Pin_5); no longer J4.5 (Pin_5)
- net at J5.2 (Pin_2): now also J6.2 (Pin_2); no longer J4.2 (Pin_2)
- net at J5.3 (Pin_3): now also J6.3 (Pin_3); no longer J4.3 (Pin_3)
Other:
- moved on the sheet: J2, J3, J5, J7, J8
Changed lines of the file:
@@
 U 1 1 616CD407
 P 6150 2450
-F 0 "J2" H 6250 2700 50  0000 C CNN
-F 1 "Conn_01x04_Male" V 6250 3100 50  0000 C CNN
+F 0 "J2" H 6258 2731 50  0000 C CNN
+F 1 "Conn_01x04_Male" V 6150 1850 50  0000 C CNN
 F 2 "Connector_JST:JST_GH_BM04B-GHS-TBT_1x04-1MP_P1.25mm_Vertical" H 6150 2450 50  0001 C CNN
 F 3 "~" H 6150 2450 50  0001 C CNN
 	1    6150 2450
-	-1   0    0    -1
+	1    0    0    -1
 $EndComp
 $Comp
@@
 U 1 1 616CE17D
 P 6500 2450
-F 0 "J3" H 6600 2700 50  0000 C CNN
-F 1 "Conn_01x04_Male" V 6600 3100 50  0000 C CNN
+F 0 "J3" H 6608 2731 50  0000 C CNN
+F 1 "Conn_01x04_Male" V 6500 1850 50  0000 C CNN
 F 2 "Connector_JST:JST_GH_BM04B-GHS-TBT_1x04-1MP_P1.25mm_Vertical" H 6500 2450 50  0001 C CNN
 F 3 "~" H 6500 2450 50  0001 C CNN
 	1    6500 2450
-	-1   0    0    -1
+	1    0    0    -1
 $EndComp
 $Comp
-L Connector:Conn_01x06_Male J4
+L Connector:Conn_01x04_Male J4
 U 1 1 616CE520
-P 7300 2450
-F 0 "J4" H 7408 2731 50  0000 C CNN
-F 1 "Conn_01x04_Male" V 7400 3150 50  0000 C CNN
-F 2 "Connector_JST:JST_GH_BM06B-GHS-TBT_1x06-1MP_P1.25mm_Vertical" H 7300 2450 50  0001 C CNN
-F 3 "~" H 7300 2450 50  0001 C CNN
-	1    7300 2450
-	-1   0    0    -1
+P 6800 2450
+F 0 "J4" H 6908 2731 50  0000 C CNN
+F 1 "Conn_01x04_Male" V 6800 1850 50  0000 C CNN
+F 2 "Connector_JST:JST_GH_BM04B-GHS-TBT_1x04-1MP_P1.25mm_Vertical" H 6800 2450 50  0001 C CNN
+F 3 "~" H 6800 2450 50  0001 C CNN
+	1    6800 2450
+	1    0    0    -1
 $EndComp
 $Comp
 L Connector:Conn_01x06_Male J5
 U 1 1 616CE858
-P 7650 2450
-F 0 "J5" H 7758 2731 50  0000 C CNN
-F 1 "Conn_01x04_Male" V 7750 3150 50  0000 C CNN
-F 2 "Connector_JST:JST_GH_BM06B-GHS-TBT_1x06-1MP_P1.25mm_Vertical" H 7650 2450 50  0001 C CNN
-F 3 "~" H 7650 2450 50  0001 C CNN
-	1    7650 2450
-	-1   0    0    -1
-$EndComp
-$Comp
-L Connector:Conn_01x02_Male J1
-U 1 1 616CEFDD
-P 5100 2450
-F 0 "J1" H 5208 2631 50  0000 C CNN
-F 1 "Conn_01x02_Male" H 5208 2540 50  0000 C CNN
-F 2 "Connector_JST:JST_GH_BM02B-GHS-TBT_1x02-1MP_P1.25mm_Vertical" H 5100 2450 50  0001 C CNN
-F 3 "~" H 5100 2450 50  0001 C CNN
-	1    5100 2450
+P 7250 2450
+F 0 "J5" H 7350 2800 50  0000 C CNN
+F 1 "Conn_01x06_Male" V 7250 1750 50  0000 C CNN
+F 2 "Connector_JST:JST_GH_BM06B-GHS-TBT_1x06-1MP_P1.25mm_Vertical" H 7250 2450 50  0001 C CNN
+F 3 "~" H 7250 2450 50  0001 C CNN
+	1    7250 2450
 	1    0    0    -1
 $EndComp
+Connection ~ 6350 2350
+Connection ~ 6700 2350
 Wire Wire Line
-	5300 2450 5650 2450
+	6700 2350 7000 2350
+Connection ~ 6350 2650
+Connection ~ 6700 2650
 Wire Wire Line
-	5650 2450 5650 2350
+	6700 2650 7000 2650
+Connection ~ 6700 2550
 Wire Wire Line
-	5650 2350 5800 2350
+	6700 2550 6350 2550
 Wire Wire Line
-	5300 2550 5650 2550
+	7000 2550 6700 2550
 Wire Wire Line
-	5650 2550 5650 2650
+	6350 2450 6700 2450
+Connection ~ 6700 2450
 Wire Wire Line
-	5650 2650 5800 2650
+	6700 2450 7000 2450
 $Comp
 L power:Earth #PWR0101
 U 1 1 616D04C1
-P 5800 2950
-F 0 "#PWR0101" H 5800 2700 50  0001 C CNN
-F 1 "Earth" H 5800 2800 50  0001 C CNN
-F 2 "" H 5800 2950 50  0001 C CNN
-F 3 "~" H 5800 2950 50  0001 C CNN
-	1    5800 2950
+P 5850 2950
+F 0 "#PWR0101" H 5850 2700 50  0001 C CNN
+F 1 "Earth" H 5850 2800 50  0001 C CNN
+F 2 "" H 5850 2950 50  0001 C CNN
+F 3 "~" H 5850 2950 50  0001 C CNN
+	1    5850 2950
 	1    0    0    -1
 $EndComp
@@
 L power:+5V #PWR0102
 U 1 1 616D0A70
-P 5800 2000
-F 0 "#PWR0102" H 5800 1850 50  0001 C CNN
-F 1 "+5V" H 5815 2173 50  0000 C CNN
-F 2 "" H 5800 2000 50  0001 C CNN
-F 3 "" H 5800 2000 50  0001 C CNN
-	1    5800 2000
+P 5950 2000
+F 0 "#PWR0102" H 5950 1850 50  0001 C CNN
+F 1 "+5V" H 5965 2173 50  0000 C CNN
+F 2 "" H 5950 2000 50  0001 C CNN
+F 3 "" H 5950 2000 50  0001 C CNN
+	1    5950 2000
 	1    0    0    -1
 $EndComp
 Wire Wire Line
-	5800 2350 5800 2100
-Connection ~ 5800 2350
-Wire Wire Line
-	5800 2350 5950 2350
-Wire Wire Line
-	5800 2650 5800 2800
-Connection ~ 5800 2650
-Wire Wire Line
-	5800 2650 5950 2650
+	5950 2350 5950 2100
 $Comp
 L Connector:Conn_01x01_Male J7
 U 1 1 616D4732
-P 5300 2100
-F 0 "J7" H 5408 2281 50  0000 C CNN
-F 1 "5V" H 5408 2190 50  0000 C CNN
-F 2 "TestPoint:TestPoint_Pad_2.5x2.5mm" H 5300 2100 50  0001 C CNN
-F 3 "~" H 5300 2100 50  0001 C CNN
-	1    5300 2100
+P 5450 2100
+F 0 "J7" H 5558 2281 50  0000 C CNN
+F 1 "5V" H 5558 2190 50  0000 C CNN
+F 2 "TestPoint:TestPoint_Pad_2.5x2.5mm" H 5450 2100 50  0001 C CNN
+F 3 "~" H 5450 2100 50  0001 C CNN
+	1    5450 2100
 	1    0    0    -1
 $EndComp
@@
 L Connector:Conn_01x01_Male J8
 U 1 1 616D4A04
-P 5300 2800
-F 0 "J8" H 5408 2981 50  0000 C CNN
-F 1 "GND" H 5408 2890 50  0000 C CNN
-F 2 "TestPoint:TestPoint_Pad_2.5x2.5mm" H 5300 2800 50  0001 C CNN
-F 3 "~" H 5300 2800 50  0001 C CNN
-	1    5300 2800
+P 5450 2800
+F 0 "J8" H 5558 2981 50  0000 C CNN
+F 1 "GND" H 5558 2890 50  0000 C CNN
+F 2 "TestPoint:TestPoint_Pad_2.5x2.5mm" H 5450 2800 50  0001 C CNN
+F 3 "~" H 5450 2800 50  0001 C CNN
+	1    5450 2800
 	1    0    0    -1
 $EndComp
 Wire Wire Line
-	5800 2950 5800 2800
+	5950 2100 5650 2100
+Connection ~ 5950 2100
 Wire Wire Line
-	5800 2800 5500 2800
-Connection ~ 5800 2800
+	5950 2100 5950 2000
+$Comp
+L Connector:Conn_01x06_Male J6
+U 1 1 616CEBB2
+P 7550 2450
+F 0 "J6" H 7650 2800 50  0000 C CNN
+F 1 "Conn_01x06_Male" V 7550 1750 50  0000 C CNN
+F 2 "Connector_JST:JST_GH_BM06B-GHS-TBT_1x06-1MP_P1.25mm_Vertical" H 7550 2450 50  0001 C CNN
+F 3 "~" H 7550 2450 50  0001 C CNN
+	1    7550 2450
+	1    0    0    -1
+$EndComp
 Wire Wire Line
-	5800 2100 5500 2100
-Connection ~ 5800 2100
+	7750 2250 7450 2250
 Wire Wire Line
-	5800 2100 5800 2000
+	7450 2250 7150 2250
 Wire Wire Line
-	6900 2350 6900 2250
+	7150 2250 7150 2350
 Wire Wire Line
-	6900 2250 7100 2250
-Connection ~ 5950 2350
-Connection ~ 5950 2650
+	7150 2350 7000 2350
+Connection ~ 7450 2250
+Connection ~ 7000 2350
 Wire Wire Line
-	5950 2350 6300 2350
+	7450 2750 7750 2750
 Wire Wire Line
-	5950 2650 6300 2650
-Connection ~ 6300 2350
+	7750 2650 7450 2650
 Wire Wire Line
-	6300 2350 6900 2350
-Connection ~ 7100 2250
+	7450 2350 7750 2350
 Wire Wire Line
-	7100 2250 7450 2250
-Connection ~ 7100 2750
+	7450 2450 7750 2450
 Wire Wire Line
-	7100 2750 7450 2750
+	7750 2550 7450 2550
 Wire Wire Line
-	6950 2450 6950 2550
+	7200 2550 7200 2450
 Wire Wire Line
-	6950 2550 7100 2550
+	7200 2450 7000 2450
+Connection ~ 7450 2550
 Wire Wire Line
-	5950 2450 6300 2450
-Connection ~ 6300 2450
+	7450 2550 7200 2550
+Connection ~ 7000 2450
 Wire Wire Line
-	6300 2450 6950 2450
-Connection ~ 7100 2550
+	7450 2650 7100 2650
 Wire Wire Line
-	7100 2550 7450 2550
+	7100 2650 7100 2550
 Wire Wire Line
-	5950 2550 6300 2550
+	7100 2550 7000 2550
+Connection ~ 7450 2650
+Connection ~ 7000 2550
 Wire Wire Line
-	6900 2550 6900 2650
+	7450 2750 7000 2750
 Wire Wire Line
-	6900 2650 7100 2650
-Connection ~ 6300 2550
+	7000 2750 7000 2650
+Connection ~ 7450 2750
+Connection ~ 7000 2650
 Wire Wire Line
-	6300 2550 6900 2550
-Connection ~ 7100 2650
+	5650 2800 5850 2800
 Wire Wire Line
-	7100 2650 7450 2650
+	5850 2800 5850 2950
 Wire Wire Line
-	6850 2750 6850 2650
+	5850 2650 5850 2800
+Connection ~ 5850 2800
 Wire Wire Line
-	6850 2650 6300 2650
+	5950 2350 6350 2350
 Wire Wire Line
-	6850 2750 7100 2750
-Connection ~ 6300 2650
+	5850 2650 6350 2650
+Connection ~ 6500 2350
+Connection ~ 6500 2650
 Wire Wire Line
-	7100 2350 7450 2350
+	6350 2350 6500 2350
 Wire Wire Line
-	7100 2450 7450 2450
+	6350 2650 6500 2650
+Wire Wire Line
+	6350 2350 6700 2350
+Wire Wire Line
+	6350 2650 6700 2650
 $EndSCHEMATC
